Commit message: Add sawyer environments

File: garage/contrib/ros/worlds/models/pnp_block/model.urdf (robot description, URDF)
Before this commit: robot block, 1 links, 0 joints
Links:
- removed link block
- added link pnp_block, mass 0.7; collision box size=0.128 0.045 0.06; visual box size=0.128 0.045 0.06
