Commit message: Update

File: garage/contrib/ros/worlds/models/pnp_block/model_green.urdf (robot description, URDF)
Before this commit: robot pnp_tray, 1 links, 0 joints
Links:
- removed link pnp_tray
- added link pnp_block_green, mass 0.01; collision box size=0.03 0.03 0.04; visual box size=0.03 0.03 0.04

File: garage/contrib/ros/worlds/models/pnp_block/model_red.urdf (robot description, URDF)
Before this commit: robot pnp_tray, 1 links, 0 joints
Links:
- removed link pnp_tray
- added link pnp_block_red, mass 0.01; collision box size=0.05 0.05 0.05; visual box size=0.05 0.05 0.05

File: garage/contrib/ros/worlds/models/pnp_block/model_yellow.urdf (robot description, URDF)
Before this commit: robot pnp_block, 1 links, 0 joints
Links:
- removed link pnp_block
- added link pnp_block_yellow, mass 0.01; collision box size=0.05 0.04 0.04; visual box size=0.05 0.04 0.04
