Commit message: rocks!

File: garage/contrib/ros/worlds/models/table/model.urdf (robot description, URDF)
Before this commit: robot pnp_block, 1 links, 0 joints
Links:
- removed link pnp_block
- added link table, mass 0.7; collision box size=1.2 1 0.1; visual box size=1.2 1 0.1

File: garage/contrib/ros/worlds/models/tray/model.urdf (robot description, URDF)
Before this commit: robot pnp_block, 1 links, 0 joints
Links:
- removed link pnp_block
- added link pnp_tray, mass 0.7; collision box size=0.10 0.10 0.008; visual box size=0.10 0.10 0.008
